Commit message: Update v1.1
- Some lidar feature changes in inota.urdf.

File: inota_description/urdf/inota.urdf (robot description, URDF)
Before this commit: robot inota, 12 links, 11 joints
Links:
- removed link camera_link
- removed link camera_rgb_frame
- removed link camera_rgb_optic_frame
- removed link lidar_link
- added link scan_link; visual mesh filename=package://inota_description/meshes/lidar.stl scale=0.001 0.001 0.001
Joints:
- removed joint camera_joint
- removed joint camera_rgb_joint
- removed joint camera_rgb_optic_joint
- removed joint lidar_joint
- added joint scan_joint: type fixed, parent base_link, child scan_link, origin xyz=-0.28 0.001 0.029 rpy=0 0 3.14

Commit message: Update v1.2
- Depth camera features added.
- Odom rotation fixed.

File: inota_description/urdf/inota.urdf (robot description, URDF)
Before this commit: robot inota, 9 links, 8 joints
Links:
- added link camera_link; visual mesh filename=package://inota_description/meshes/camera.stl scale=0.001 0.001 0.001
- added link camera_rgb_frame
- added link camera_rgb_optic_frame
Joints:
- added joint camera_joint: type fixed, parent base_link, child camera_link, origin xyz=0.36 0.001 0.0795 rpy=0 0 0
- added joint camera_rgb_joint: type fixed, parent camera_link, child camera_rgb_frame, origin xyz=0 0 0 rpy=0 0 0
- added joint camera_rgb_optic_joint: type fixed, parent camera_rgb_frame, child camera_rgb_optic_frame, origin xyz=0 0 0 rpy=0 0 0
- joint left_wheel_joint: axis 0 -1 0 -> 0 1 0; origin xyz=0 -0.22 -0.052 rpy=0.0 0.0 0.0 -> xyz=0 0.22 -0.052 rpy=0 0 0
- joint right_wheel_joint: axis 0 -1 0 -> 0 1 0; origin xyz=0 0.22 -0.052 rpy=0 0 0 -> xyz=0 -0.22 -0.052 rpy=0.0 0.0 0.0
- joint scan_joint: origin xyz=-0.28 0.001 0.029 rpy=0 0 3.14 -> xyz=0.28 0.001 0.029 rpy=0 0 0

Commit message: Update v1.3
- Some URDF fixes.

File: inota_description/urdf/inota.urdf (robot description, URDF)
Before this commit: robot inota, 12 links, 11 joints
Links:
- link base_link: geometry collision mesh filename=package://inota_description/meshes/inota.stl scale=0.001 0.001 0.001; visual mesh filename=package://inota_description/meshes/inota.stl scale=0.001 0.001 0.001
